File: EAGLE/PCB_PIC24_CARD/pic24_card.sch (EAGLE design)
At the start: 25 parts, among them IC1 PIC24FJ256GL410, IC2 XR3072XID-F, M1 MOUNTING_3M_3.2MM, X1 CONN_SMD_67P-P0.5-V_NASB0-S67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, X2 M.2_MKEY_FINGERS, X3 5-PIN_2.54_HEADER

Commit message: pic24 card is done, gerbers and jlc files generated
Parts:
- added R8: 470R, _NIBE_rcl:R-EU_R0402_NIBE
- added STATUS: LED_YELLOW, _NIBE_rcl:R-EU_R0603
Connections:
- removed net N$10: X1.59, X2.16
- removed net N$100: IC1_REMAPPABLE.RPI45/RF1
- removed net N$101: IC1_ANALOG.AN2/RP13/RB2
- removed net N$102: IC1_ANALOG.AN3/RB3
- removed net N$103: IC1_ANALOG.AN4/RP28/RB4
- removed net N$104: IC1_ANALOG.AN5/RP18/RB5
- removed net N$105: IC1_ANALOG.AN6/RP6/RB6
- removed net N$106: IC1_ANALOG.AN7/RP7/RB7
- removed net N$107: IC1_ANALOG.AN8/RP8/RB8
- removed net N$108: IC1_ANALOG.AN9/RP9/RB9
- removed net N$109: IC1_ANALOG.AN10/RPI44/RB10
- removed net N$11: X1.57, X2.18
- removed net N$110: IC1_ANALOG.AN11RB11
- removed net N$111: IC1_ANALOG.AN12/RB12
- removed net N$112: IC1_ANALOG.AN13/RB13
- removed net N$113: IC1_ANALOG.AN14/RP14/RB14
- removed net N$114: IC1_ANALOG.AN15/RP29/RB15
- removed net N$115: IC1_ANALOG.AN16/RPI41/RC4
- removed net N$116: IC1_ANALOG.AN17/RP21/RG6
- removed net N$117: IC1_ANALOG.AN18/RP6/RG7
- removed net N$118: IC1_ANALOG.AN19/RP19/RG8
- removed net N$119: IC1_ANALOG.AN20/RP27/RG9
- removed net N$12: X1.55, X2.20
- removed net N$120: IC1_ANALOG.AN21/RPI48/RE9
- removed net N$121: IC1_ANALOG.AN22/RA6
- removed net N$122: IC1_ANALOG.AN23/RA7
- removed net N$13: X1.53, X2.22
- removed net N$14: X1.51, X2.24
- removed net N$15: X1.21, X2.54
- removed net N$16: X1.27, X2.48
- removed net N$17: X1.29, X2.46
- removed net N$18: X1.31, X2.44
- removed net N$19: X1.33, X2.42
- removed net N$2: X1.25, X2.50
- removed net N$20: X1.35, X2.40
- removed net N$21: X1.37, X2.38
- removed net N$22: X1.39, X2.36
- removed net N$23: X1.41, X2.34
- removed net N$24: X1.43, X2.32
- removed net N$25: X1.45, X2.30
- removed net N$26: X1.47, X2.28
- removed net N$27: X1.49, X2.26
- removed net N$28: X1.11, X2.56
- removed net N$29: X1.9, X2.58
- removed net N$3: X1.73, X2.2
- removed net N$33: X1.2, X2.75
- removed net N$34: X1.22, X2.55
- removed net N$35: X1.4, X2.73
- removed net N$4: X1.71, X2.4
- removed net N$40: X1.24, X2.53
- removed net N$41: X1.26, X2.51
- removed net N$42: X1.28, X2.49
- removed net N$43: X1.30, X2.47
- removed net N$44: X1.32, X2.45
- removed net N$45: X1.34, X2.43
- removed net N$46: X1.36, X2.41
- removed net N$47: X1.38, X2.39
- removed net N$48: X1.40, X2.37
- removed net N$49: X1.42, X2.35
- removed net N$5: X1.69, X2.6
- removed net N$50: X1.44, X2.33
- removed net N$51: X1.74, X2.3
- removed net N$52: X1.72, X2.5
- removed net N$53: X1.70, X2.7
- removed net N$54: X1.68, X2.9
- removed net N$55: X1.66, X2.11
- removed net N$56: X1.64, X2.13
- removed net N$57: X1.62, X2.15
- removed net N$58: X1.60, X2.17
- removed net N$59: X1.58, X2.19
- removed net N$6: X1.67, X2.8
- removed net N$60: X1.56, X2.21
- removed net N$61: X1.54, X2.23
- removed net N$62: X1.52, X2.25
- removed net N$63: X1.46, X2.31
- removed net N$64: X1.48, X2.29
- removed net N$65: X1.50, X2.27
- removed net N$68: IC1_REMAPPABLE.RP34/RE5
- removed net N$69: IC1_REMAPPABLE.RP35/SCL3/RE6
- removed net N$7: X1.65, X2.10
- removed net N$70: IC1_REMAPPABLE.RP36/SDA3/RE7
- removed net N$72: IC1_REMAPPABLE.RP5/RD15
- removed net N$73: IC1_REMAPPABLE.RP10/RF4
- removed net N$74: IC1_REMAPPABLE.RP17/RF5
- removed net N$75: IC1_REMAPPABLE.RP16/RF3
- removed net N$76: IC1_REMAPPABLE.RP30/RF2
- removed net N$77: IC1_REMAPPABLE.RP15/RF8
- removed net N$78: IC1_REMAPPABLE.RP2/RD8
- removed net N$79: IC1_REMAPPABLE.RP4/RD9
- removed net N$8: X1.63, X2.12
- removed net N$80: IC1_REMAPPABLE.RP3/RD10
- removed net N$81: IC1_REMAPPABLE.RP12/RD11
- removed net N$82: IC1_REMAPPABLE.RP11/RD0
- removed net N$83: IC1_REMAPPABLE.RP23/RD2
- removed net N$84: IC1_REMAPPABLE.RP24/RD1
- removed net N$85: IC1_REMAPPABLE.RP22/RD3
- removed net N$86: IC1_REMAPPABLE.RP25/SDI3/RD4
- removed net N$87: IC1_REMAPPABLE.RP20/SD03/RD5
- removed net N$88: IC1_REMAPPABLE.RP32/RD6
- removed net N$89: IC1_REMAPPABLE.RP33/RD7
- removed net N$9: X1.61, X2.14
- removed net N$90: IC1_REMAPPABLE.RPI38/RC1
- removed net N$91: IC1_REMAPPABLE.RPI39/RC2
- removed net N$92: IC1_REMAPPABLE.RPI40/RC3
- removed net N$93: IC1_REMAPPABLE.RPI47/RE8
- removed net N$95: IC1_REMAPPABLE.RPI43/RD14
- removed net N$96: IC1_REMAPPABLE.RPI50/RA14
- removed net N$97: IC1_REMAPPABLE.RPI49/RA15
- removed net N$98: IC1_REMAPPABLE.RPI37/RC14
- removed net N$99: IC1_REMAPPABLE.RPI42/RD12
- new net AN10: IC1_ANALOG.AN10/RPI44/RB10, X1.47, X2.28
- new net AN11: IC1_ANALOG.AN11RB11, X1.58, X2.19
- new net AN12: IC1_ANALOG.AN12/RB12, X1.45, X2.30
- new net AN13: IC1_ANALOG.AN13/RB13, X1.43, X2.32
- new net AN14: IC1_ANALOG.AN14/RP14/RB14, X1.56, X2.21
- new net AN15: IC1_ANALOG.AN15/RP29/RB15, X1.50, X2.27
- new net AN16: IC1_ANALOG.AN16/RPI41/RC4, X1.57, X2.18
- new net AN17: IC1_ANALOG.AN17/RP21/RG6, X1.64, X2.13
- new net AN18: IC1_ANALOG.AN18/RP6/RG7, X1.59, X2.16
- new net AN19: IC1_ANALOG.AN19/RP19/RG8, X1.61, X2.14
- new net AN2: IC1_ANALOG.AN2/RP13/RB2, X1.70, X2.7
- new net AN20: IC1_ANALOG.AN20/RP27/RG9, X1.66, X2.11
- new net AN21: IC1_ANALOG.AN21/RPI48/RE9, X1.65, X2.10
- new net AN22: IC1_ANALOG.AN22/RA6, X1.52, X2.25
- new net AN23: IC1_ANALOG.AN23/RA7, X1.54, X2.23
- new net AN3: IC1_ANALOG.AN3/RB3, X1.69, X2.6
- new net AN4: IC1_ANALOG.AN4/RP28/RB4, X1.67, X2.8
- new net AN5: IC1_ANALOG.AN5/RP18/RB5, X1.68, X2.9
- new net AN6: IC1_ANALOG.AN6/RP6/RB6, X1.71, X2.4
- new net AN7: IC1_ANALOG.AN7/RP7/RB7, X1.72, X2.5
- new net AN8: IC1_ANALOG.AN8/RP8/RB8, X1.60, X2.17
- new net AN9: IC1_ANALOG.AN9/RP9/RB9, X1.49, X2.26
- new net LED_STATUS: IC1_DIGITAL.RF7, R8.1
- new net RC13: IC1_DIGITAL.RC13, X1.22, X2.55
- new net RP10: IC1_REMAPPABLE.RP10/RF4, X1.35, X2.40
- new net RP11: IC1_REMAPPABLE.RP11/RD0, X1.36, X2.41
- new net RP12: IC1_REMAPPABLE.RP12/RD11, X1.34, X2.43
- new net RP15: IC1_REMAPPABLE.RP15/RF8, X1.27, X2.48
- new net RP16: IC1_REMAPPABLE.RP16/RF3, X1.31, X2.44
- new net RP17: IC1_REMAPPABLE.RP17/RF5, X1.33, X2.42
- new net RP2: IC1_REMAPPABLE.RP2/RD8, X1.28, X2.49
- new net RP20: IC1_REMAPPABLE.RP20/SD03/RD5, X1.21, X2.54
- new net RP22: IC1_REMAPPABLE.RP22/RD3, X1.44, X2.33
- new net RP23: IC1_REMAPPABLE.RP23/RD2, X1.42, X2.35
- new net RP24: IC1_REMAPPABLE.RP24/RD1, X1.40, X2.37
- new net RP25: IC1_REMAPPABLE.RP25/SDI3/RD4, X1.48, X2.29
- new net RP3: IC1_REMAPPABLE.RP3/RD10, X1.32, X2.45
- new net RP30: IC1_REMAPPABLE.RP30/RF2, X1.29, X2.46
- new net RP32: IC1_REMAPPABLE.RP32/RD6, X1.23, X2.52
- new net RP33: IC1_REMAPPABLE.RP33/RD7, X1.25, X2.50
- new net RP34: IC1_REMAPPABLE.RP34/RE5, X1.51, X2.24
- new net RP35: IC1_REMAPPABLE.RP35/SCL3/RE6, X1.73, X2.2
- new net RP36: IC1_REMAPPABLE.RP36/SDA3/RE7, X1.74, X2.3
- new net RP4: IC1_REMAPPABLE.RP4/RD9, X1.30, X2.47
- new net RP5: IC1_REMAPPABLE.RP5/RD15, X1.37, X2.38
- new net RPI37: IC1_REMAPPABLE.RPI37/RC14, X1.38, X2.39
- new net RPI38: IC1_REMAPPABLE.RPI38/RC1, X1.53, X2.22
- new net RPI39: IC1_REMAPPABLE.RPI39/RC2, X1.62, X2.15
- new net RPI40: IC1_REMAPPABLE.RPI40/RC3, X1.55, X2.20
- new net RPI42: IC1_REMAPPABLE.RPI42/RD12, X1.46, X2.31
- new net RPI43: IC1_REMAPPABLE.RPI43/RD14, X1.39, X2.36
- new net RPI45: IC1_REMAPPABLE.RPI45/RF1, X1.41, X2.34
- new net RPI47: IC1_REMAPPABLE.RPI47/RE8, X1.63, X2.12
- new net RPI49: IC1_REMAPPABLE.RPI49/RA15, X1.26, X2.51
- new net RPI50: IC1_REMAPPABLE.RPI50/RA14, X1.24, X2.53
- net A: now also X1.9, X2.58
- net B: now also X1.11, X2.56
- net GND: now also STATUS.2, X1.2, X1.4, X2.73, X2.75
- net N$1: now also R8.2, STATUS.1; no longer X1.23, X2.52
