File: EAGLE/PCB_PWR_SUPPLY_CARD/power_supply_card.brd (EAGLE design)
At the start: 24 x 60 mm, 5 parts, among them M1 MOUNTING_3M_3.2MM, X1 CONN_SMD_67P-P0.5-V_NASB0-S67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, X2 M.2_MKEY_FINGERS

Commit message: finish pwr supply card
Parts:
- added C1: RXW221M1JBK-1020, Enertech_Capacitor:THROUGH_HOLE_5.0P_10MMD
- added C10: 150n, _NIBE_rcl:C0603
- added C11, C4, C9: 100n 50V, _NIBE_rcl:C0603
- added C12: 150n, _NIBE_rcl:C0402_NIBE
- added C13, C14: 10u, _NIBE_rcl:C0603
- added C3: 4u7 100V, _NIBE_rcl:C1210
- added C5, C6, C7, C8: 10u 50V, _NIBE_rcl:C1210
- added D1: RS1J, _NIBE_DIODES:DO-214AC(SMA)
- added D2, D3: DSS16U, Enertech_Diode:SOD123F
- added IC1: LIN_REG_ADJ_SOT223, ENERTECH_MISC:SOT223
- added L1: 10u, _NIBE_rcl:L4532P
- added L2: 100u, Enertech_Inductor:ASPI-8040S
- added L3: 74404063470, Enertech_Inductor:74404063470
- added R1: B72520T0400K062, _NIBE_rcl:R1206
- added R3: 2R 1W, _NIBE_rcl:R2512
- added R4, R7: 47k, _NIBE_rcl:R0402_NIBE
- added R5: 22k, _NIBE_rcl:R0402_NIBE
- added R6: 200k, _NIBE_rcl:R0402_NIBE
- added R8: 130k, _NIBE_rcl:R0402_NIBE
- added R9: 220k, _NIBE_rcl:R0402_NIBE
- added U1, U2: ST1S14PHR, ST1S14PHR:HSOP8_STM
- added X3: 1751248, con-phoenix-350:1751248
Connections:
- removed net N$30: X1.P$7, X2.68
- removed net N$31: X1.P$5, X2.70
- removed net N$36: X1.P$6, X2.71
- removed net N$37: X1.P$8, X2.69
- removed net N$38: X1.P$10, X2.67
- removed net N$39: X1.P$20, X2.57
- new net +12V: C10.2, C13.1, C6.1, IC1.3, L2.P$2, R4.1, R6.2, X1.P$5, X2.70
- new net N$34: D1.K, R3.1
- new net N$35: C1.1, C3.1, L1.1, R3.2
- new net N$40: R4.2, U1.2
- new net N$41: C9.1, U1.1
- new net N$42: C9.2, D2.1, L2.P$1, U1.8
- new net N$43: C10.1, R5.1, R6.1, U1.4
- new net N$45: C11.1, U2.1
- new net N$46: C11.2, D3.1, L3.P$1, U2.8
- new net N$47: R7.1, U2.2
- new net N$48: C12.1, R8.2, R9.2, U2.4
- new net R: D1.A, R1.2, X1.P$10, X1.P$20, X1.P$6, X1.P$7, X1.P$8, X2.57, X2.67, X2.68, X2.69, X2.71, X3.1
- new net R_RECT: C4.1, C5.1, C7.1, L1.2, U1.5, U1.7, U2.5, U2.7
- net +3V3: now also C12.2, C8.1, L3.P$2, R7.2, R9.1
- net +5V: now also C14.1, IC1.1, IC1.4
- net GND: now also C1.2, C13.2, C14.2, C3.2, C4.2, C5.2, C6.2, C7.2, C8.2, D2.2, D3.2, IC1.2, R1.1, R5.2, R8.1, U1.3, U1.6, U1.EPAD, U2.3, U2.6, U2.EPAD, X3.2
Routing:
- net +12V: track 0.00 -> 58.6 mm, vias 0 -> 3
- net GND: track 8.77 -> 27.4 mm, vias 4 -> 25
- net R: track 0.00 -> 15.2 mm, vias 0 -> 5
- net N$36: track 13.3 -> 0.00 mm
- net N$37: track 13.3 -> 0.00 mm
- net N$38: track 13.3 -> 0.00 mm
- net N$31: track 11.6 -> 0.00 mm, vias 1 -> 0
- net N$30: track 11.4 -> 0.00 mm, vias 1 -> 0
- net +5V: track 15.7 -> 23.4 mm, vias 1 -> 5
- net N$39: track 4.45 -> 0.00 mm
- net +3V3: track 7.17 -> 10.3 mm, vias 3 -> 7
- added copper zone on layer 1, net +12V
- added copper zone on layer 1, net +3V3
- added copper zone on layer 1, net +5V
- added copper zone on layer 16, net +5V
- added copper zone on layer 1, net N$34
- added copper zone on layer 1, net N$35
- added copper zone on layer 1, net N$40
- added copper zone on layer 1, net N$41
- added copper zone on layer 1, net N$42
- added copper zone on layer 1, net N$43
- added copper zone on layer 1, net N$45
- added copper zone on layer 1, net N$46
- added copper zone on layer 1, net N$47
- added copper zone on layer 1, net N$48
- added copper zone on layer 1, net R
- added copper zone on layer 16, net R
- added copper zone on layer 1, net R_RECT
